Commit message: added second servo

File: urdf/robby_track2.urdf (robot description, URDF)
Before this commit: robot robby_track2, 3 links, 2 joints
Links:
- added link servo2_head; visual box size=0.1 .1 .05
- link base_link: geometry visual box size=0.3 0.15 0.05
- link servo1_base: geometry visual box size=0.03 0.02 0.05
- link servo1_head: geometry visual box size=0.05 .05 .05
Joints:
- added joint servo1_to_servo2: type continuous, parent servo1_head, child servo2_head, origin xyz=0.0 0 0.1 rpy=0 0 0, axis 0 1 0
- joint servo1_base_to_head: origin xyz=0 0 0.01 rpy=0 0 0 -> xyz=0.1 0 0.05 rpy=0 0 0; parent base_link -> servo1_base

Commit message: urdf and state_publisher now correct, cleanup of arduino

File: urdf/robby_track2.urdf (robot description, URDF)
Before this commit: robot robby_track2, 4 links, 3 joints
Links:
- added link ultraSonic; visual box size=0.02 0.05 0.02
- link base_link: geometry visual box size=0.2 0.105 0.075
- link servo1_base: geometry visual box size=0.02 0.01 0.03
- link servo1_head: geometry visual box size=0.03 0.05 0.03
- link servo2_head: geometry visual box size=0.03 0.05 0.03
Joints:
- removed joint servo1_base_to_head
- added joint base_to_head1: type continuous, parent base_link, child servo1_head, origin xyz=0.095 0 0.0675 rpy=0 0 0, axis 0 0 1
- added joint servo1_to_ultraSonic: type fixed, parent servo1_head, child ultraSonic, origin xyz=0.035 0.0 -0.01 rpy=0 0 0, axis 0 1 0
- joint base_to_servo1: origin (none) -> xyz=0 0 0 rpy=0 0 0
- joint servo1_to_servo2: origin xyz=0.0 0 0.1 rpy=0 0 0 -> xyz=0.0 0.0 0.03 rpy=0 0 0

Commit message: added real_sense camera to rviz

File: urdf/robby_track2.urdf (robot description, URDF)
Before this commit: robot robby_track2, 5 links, 4 joints
Links:
- added link camera_link; visual box size=0.010 0.130 0.019
Joints:
- added joint servo2_to_camera_link: type fixed, parent servo2_head, child camera_link, origin xyz=0.035 -0.045 0.0 rpy=0 0 0, axis 0 1 0

Commit message: moved servo control to state publisher

File: urdf/robby_track2.urdf (robot description, URDF)
Before this commit: robot robby_track2, 6 links, 5 joints
Joints:
- joint base_to_head1: origin xyz=0.095 0 0.0675 rpy=0 0 0 -> xyz=0.095 0 0.105 rpy=0 0 0

Commit message: BNO055 added to urdf and robot_localisation

File: urdf/robby_track2.urdf (robot description, URDF)
Before this commit: robot robby_track2, 6 links, 5 joints
Links:
- added link imu; visual box size=0.003 0.005 0.001
- added link imu_base; visual box size=0.067 0.052 0.023
Joints:
- added joint base_to_imu: type fixed, parent base_link, child imu, origin xyz=0.0335 0 0.0985 rpy=0 0 -1.5707963268
- added joint base_to_imu_base: type fixed, parent base_link, child imu_base, origin xyz=0 0 0 rpy=0 0 0
